File: hardware/arcticvideo.kicad_sch (KiCad schematic)
At the start: 0 parts

Commit message: last commit for a while, i have to change the fpga and i dont have the time, money, or motivation to do that
Other:
- added sheet fpga1 (fpga1.kicad_sch)
Changed lines of the file:
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@@
+	)
+	(sheet
+		(at 185.42 73.66)
+		(size 81.28 52.07)
+		(exclude_from_sim no)
+		(in_bom yes)
+		(on_board yes)
+		(dnp no)
+		(fields_autoplaced yes)
+		(stroke
+			(width 0.1524)
+			(type solid)
+		)
+		(fill
+			(color 0 0 0 0)
+		)
+		(property "Sheetname" "fpga1"
+			(at 185.42 72.9484 0)
+			(show_name no)
+			(do_not_autoplace no)
+			(effects
+				(font
+					(size 1.27 1.27)
+				)
+				(justify left bottom)
+			)
+		)
+		(property "Sheetfile" "fpga1.kicad_sch"
+			(at 185.42 126.3146 0)
+			(show_name no)
+			(do_not_autoplace no)
+			(effects
+				(font
+					(size 1.27 1.27)
+				)
+				(justify left top)
+			)
+		)
+		(instances
+			(project "arcticvideo"
+				(path "/9e9873e7-449f-4340-a6d8-702e1fa8c41f"
+					(page "8")
+				)
+			)
+		)
 	)
 	(sheet
