File: hardware/fpga.kicad_sch (KiCad schematic)
At the start: 0 parts

Commit message: last commit for a while, i have to change the fpga and i dont have the time, money, or motivation to do that
Parts:
- added U? (x4): XC7A35T-2FGG484C, FGG484_AMD, symbol arcticvideo:XC7A35T-2FGG484C
- added U? (x2): XC7A75T-2FGG484C, FGG484ARTIX-7_AMD, symbol arcticvideo:XC7A75T-2FGG484C
Connections:
- new net *CAS: U?.H4 (IO_L12P_T1_MRCC_35), U?.H4 (IO_L12P_T1_MRCC_35)
- new net *CK: U?.D1 (IO_L3N_T0_DQS_AD5N_35), U?.D1 (IO_L3N_T0_DQS_AD5N_35)
- new net *CS: U?.M1 (IO_L15P_T2_DQS_35), U?.M1 (IO_L15P_T2_DQS_35)
- new net *LDQS: U?.P4 (IO_L21N_T3_DQS_35)
- new net *RAS: U?.G3 (IO_L11N_T1_SRCC_35), U?.G3 (IO_L11N_T1_SRCC_35)
- new net *RESET: U?.K4 (IO_L13P_T2_MRCC_35), U?.K4 (IO_L13P_T2_MRCC_35)
- new net *UDQS: U?.R2 (IO_L3N_T0_DQS_34), U?.R2 (IO_L3N_T0_DQS_34)
- new net *WE: U?.G4 (IO_L12N_T1_MRCC_35), U?.G4 (IO_L12N_T1_MRCC_35)
- new net A0: U?.J2 (IO_L9N_T1_DQS_AD7N_35), U?.J2 (IO_L9N_T1_DQS_AD7N_35)
- new net A1: U?.K2 (IO_L9P_T1_DQS_AD7P_35), U?.K2 (IO_L9P_T1_DQS_AD7P_35)
- new net A10/AP: U?.E2 (IO_L4P_T0_35), U?.E2 (IO_L4P_T0_35)
- new net A11: U?.B2 (IO_L2N_T0_AD12N_35), U?.B2 (IO_L2N_T0_AD12N_35)
- new net A12/*BC: U?.C2 (IO_L2P_T0_AD12P_35), U?.C2 (IO_L2P_T0_AD12P_35)
- new net A13: U?.A1 (IO_L1N_T0_AD4N_35), U?.A1 (IO_L1N_T0_AD4N_35)
- new net A14: U?.B1 (IO_L1P_T0_AD4P_35), U?.B1 (IO_L1P_T0_AD4P_35)
- new net A2: U?.G2 (IO_L8N_T1_AD14N_35), U?.G2 (IO_L8N_T1_AD14N_35)
- new net A3: U?.H2 (IO_L8P_T1_AD14P_35), U?.H2 (IO_L8P_T1_AD14P_35)
- new net A4: U?.J1 (IO_L7N_T1_AD6N_35), U?.J1 (IO_L7N_T1_AD6N_35)
- new net A5: U?.K1 (IO_L7P_T1_AD6P_35), U?.K1 (IO_L7P_T1_AD6P_35)
- new net A6: U?.F3 (IO_L6P_T0_35), U?.F3 (IO_L6P_T0_35)
- new net A7: U?.F1 (IO_L5N_T0_AD13N_35), U?.F1 (IO_L5N_T0_AD13N_35)
- new net A8: U?.G1 (IO_L5P_T0_AD13P_35), U?.G1 (IO_L5P_T0_AD13P_35)
- new net A9: U?.D2 (IO_L4N_T0_35), U?.D2 (IO_L4N_T0_35)
- new net BA0: U?.H3 (IO_L11P_T1_SRCC_35), U?.H3 (IO_L11P_T1_SRCC_35)
- new net BA1: U?.H5 (IO_L10N_T1_AD15N_35), U?.H5 (IO_L10N_T1_AD15N_35)
- new net BA2: U?.J5 (IO_L10P_T1_AD15P_35), U?.J5 (IO_L10P_T1_AD15P_35)
- new net CK: U?.E1 (IO_L3P_T0_DQS_AD5P_35), U?.E1 (IO_L3P_T0_DQS_AD5P_35)
- new net CKE: U?.L1 (IO_L15N_T2_DQS_35), U?.L1 (IO_L15N_T2_DQS_35)
- new net CLK25MHz: U?.W20 (IO_L12N_T1_MRCC_14), U?.W20 (IO_L12N_T1_MRCC_14)
- new net CLK_REF_P: U?.V4 (IO_L12P_T1_MRCC_34), U?.V4 (IO_L12P_T1_MRCC_34)
- new net CS#: U?.T19 (IO_L6P_T0_FCS_B_14), U?.T19 (IO_L6P_T0_FCS_B_14)
- new net DQ0: U?.R1 (IO_L20P_T3_35)
- new net DQ1: U?.P1 (IO_L20N_T3_35)
- new net DQ10: U?.V2 (IO_L2N_T0_34), U?.V2 (IO_L2N_T0_34)
- new net DQ11: U?.W2 (IO_L4P_T0_34), U?.W2 (IO_L4P_T0_34)
- new net DQ12: U?.Y2 (IO_L4N_T0_34), U?.Y2 (IO_L4N_T0_34)
- new net DQ13: U?.W1 (IO_L5P_T0_34), U?.W1 (IO_L5P_T0_34)
- new net DQ14: U?.Y1 (IO_L5N_T0_34), U?.Y1 (IO_L5N_T0_34)
- new net DQ15: U?.U3 (IO_L6P_T0_34), U?.U3 (IO_L6P_T0_34)
- new net DQ2: U?.P2 (IO_L22P_T3_35)
- new net DQ3: U?.N2 (IO_L22N_T3_35)
- new net DQ4: U?.M6 (IO_L23P_T3_35)
- new net DQ5: U?.M5 (IO_L23N_T3_35)
- new net DQ6: U?.P6 (IO_L24P_T3_35)
- new net DQ7: U?.N5 (IO_L24N_T3_35)
- new net DQ8: U?.U1 (IO_L1N_T0_34), U?.U1 (IO_L1N_T0_34)
- new net DQ9: U?.U2 (IO_L2P_T0_34), U?.U2 (IO_L2P_T0_34)
- new net HOLD#: U?.R21 (IO_L2N_T0_D03_14), U?.R21 (IO_L2N_T0_D03_14)
- new net LDM: U?.N4 (IO_L19P_T3_35)
- new net LDQS: U?.P5 (IO_L21P_T3_DQS_35)
- new net ODT: U?.M3 (IO_L16P_T2_35), U?.M3 (IO_L16P_T2_35)
- new net SPI_MISO: U?.R22 (IO_L1N_T0_D01_DIN_14), U?.R22 (IO_L1N_T0_D01_DIN_14)
- new net SPI_MOSI: U?.P22 (IO_L1P_T0_D00_MOSI_14), U?.P22 (IO_L1P_T0_D00_MOSI_14)
- new net SYS_CLK_P: U?.L3 (IO_L14P_T2_SRCC_35), U?.L3 (IO_L14P_T2_SRCC_35)
- new net UDM: U?.T1 (IO_L1P_T0_34), U?.T1 (IO_L1P_T0_34)
- new net UDQS: U?.R3 (IO_L3P_T0_DQS_34), U?.R3 (IO_L3P_T0_DQS_34)
- new net WP#: U?.P21 (IO_L2P_T0_D02_14), U?.P21 (IO_L2P_T0_D02_14)

Commit message: finished schematic!!! :D (before peer review)
Parts:
- removed U? (x4): XC7A35T-2FGG484C, FGG484_AMD, symbol arcticvideo:XC7A35T-2FGG484C
- removed U? (x2): XC7A75T-2FGG484C, FGG484ARTIX-7_AMD, symbol arcticvideo:XC7A75T-2FGG484C
- added U1: XC7A75T-FGG676, symbol FPGA_Xilinx_Artix7:XC7A75T-FGG676
Connections:
- net CLK25MHz: now also U1.U22 (IO_L12P_T1_MRCC_13)
- net CS#: now also U1.AB25 (IO_L7N_T1_13)
- net HOLD#: now also U1.AA25 (IO_L5N_T0_13)
- net SPI_MISO: now also U1.AA24 (IO_L7P_T1_13)
- net SPI_MOSI: now also U1.V26 (IO_L2P_T0_13)
- net WP#: now also U1.Y25 (IO_L5P_T0_13)
- new net AUX_N: U1.V16 (IO_L24P_T3_13)
- new net AUX_P: U1.V14 (IO_L23N_T3_13)
- new net DX_SEL_MONITOR: U1.V17 (IO_L24N_T3_13)
- new net HPD: U1.U14 (IO_L23P_T3_13)
- new net PERST: U1.U17 (IO_25_13)
- new net VCCOB12: U1.AA21 (VCCO_12), U1.AB18 (VCCO_12), U1.AD22 (VCCO_12), U1.AE19 (VCCO_12), U1.AF26 (VCCO_12), U1.W17 (VCCO_12)
- new net VCCOB13: U1.AC25 (VCCO_13), U1.T16 (VCCO_13), U1.T26 (VCCO_13), U1.U23 (VCCO_13), U1.V20 (VCCO_13), U1.Y24 (VCCO_13)
- new net VCCOB14: U1.K24 (VCCO_14), U1.L21 (VCCO_14), U1.N15 (VCCO_14), U1.N25 (VCCO_14), U1.P22 (VCCO_14), U1.R19 (VCCO_14)
- new net VCCOB15: U1.F26 (VCCO_15), U1.G23 (VCCO_15), U1.H20 (VCCO_15), U1.J17 (VCCO_15), U1.K14 (VCCO_15), U1.M18 (VCCO_15)
- new net VCCOB16: U1.A21 (VCCO_16), U1.B18 (VCCO_16), U1.C25 (VCCO_16), U1.D22 (VCCO_16), U1.E19 (VCCO_16), U1.F16 (VCCO_16)
- new net VCCOB33: U1.AA1 (VCCO_33), U1.AC5 (VCCO_33), U1.AD2 (VCCO_33), U1.U3 (VCCO_33), U1.W7 (VCCO_33), U1.Y4 (VCCO_33)
Other:
- note added: "can move to any io pin based on need :3"
