File: hardware/fpga.kicad_sch (KiCad schematic)
At the start: 1 part, among them U1 XC7A75T-FGG676

Commit message: pcb routing
Parts:
- U1: footprint (none) -> Package_BGA:Xilinx_FGG676
Changed lines of the file:
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@@
 			)
 		)
-		(property "Footprint" ""
+		(property "Footprint" "Package_BGA:Xilinx_FGG676"
 			(at 67.31 120.65 0)
 			(hide yes)
@@
 			)
 		)
-		(property "Footprint" ""
+		(property "Footprint" "Package_BGA:Xilinx_FGG676"
 			(at 215.9 120.65 0)
 			(hide yes)
@@
 			)
 		)
-		(property "Footprint" ""
+		(property "Footprint" "Package_BGA:Xilinx_FGG676"
 			(at 365.76 120.65 0)
 			(hide yes)
