File: hardware/clock.kicad_sch (KiCad schematic)
At the start: 1 part

Commit message: last commit for a while, i have to change the fpga and i dont have the time, money, or motivation to do that
Parts:
- added C108: 1u, symbol Device:C
- added C109, C110: 0.1u, symbol Device:C
- added R23: 22, symbol Device:R
- added XTAL2: SX3M100.000B20F30TNN, SG-210STF_EPS, symbol arcticvideo:SX3M100.000B20F30TNN
Connections:
- net +3V3: now reaches XTAL1.1
- net +3V3: now also XTAL1.4, C108.2, C109.2, C110.2, XTAL2.1 (*ST), XTAL2.4 (VCC)
- net GND: now reaches XTAL1.2
- net GND: now also C108.1, C109.1, C110.1, XTAL2.2 (GND)
- net at XTAL1.3: now also R23.2
- new net CLK25MHz: R23.1
- new net CLK_REF_P: XTAL2.3 (OUT)

Commit message: readable changes
Parts:
- removed C110: 0.1u, symbol Device:C
- added C133: 0.1u, symbol Device:C
- renumbered C108 to C131, C109 to C132, R23 to R49
Connections:
- net +3V3: now also C133.1
- net GND: now also C133.2

Commit message: pcb routing
Parts:
- C131, C132, C133: footprint (none) -> Capacitor_SMD:C_0402_1005Metric
- R47: renamed from R49; footprint (none) -> Resistor_SMD:R_0402_1005Metric
- XTAL1: footprint CHIP_ASE-24_ABR -> arcticvideo:CHIP_ASE-24_ABR
- XTAL2: footprint SG-210STF_EPS -> arcticvideo:SG-210STF_EPS
Changed lines of the file:
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@@
 		(dnp no)
 		(fields_autoplaced yes)
-		(property "Reference" "R49"
+		(property "Reference" "R47"
 			(at 123.19 86.3599 0)
 			(show_name no)
@@
 			)
 		)
-		(property "Footprint" ""
+		(property "Footprint" "Resistor_SMD:R_0402_1005Metric"
 			(at 122.428 87.63 90)
 			(hide yes)
@@
 			(project "arcticvideo"
 				(path "/9e9873e7-449f-4340-a6d8-702e1fa8c41f/c3f70c33-0f2d-4a7e-8d0b-73a0e9183494"
-					(reference "R49")
+					(reference "R47")
 					(unit 1)
 				)
@@
 			)
 		)
-		(property "Footprint" "CHIP_ASE-24_ABR"
+		(property "Footprint" "arcticvideo:CHIP_ASE-24_ABR"
 			(at 97.79 78.74 0)
 			(hide yes)
@@
 		(dnp no)
 		(fields_autoplaced yes)
-		(property "Reference" "#PWR0117"
+		(property "Reference" "#PWR0114"
 			(at 237.49 71.12 0)
 			(hide yes)
@@
 			(project "arcticvideo"
 				(path "/9e9873e7-449f-4340-a6d8-702e1fa8c41f/c3f70c33-0f2d-4a7e-8d0b-73a0e9183494"
-					(reference "#PWR0117")
+					(reference "#PWR0114")
 					(unit 1)
 				)
@@
 		(dnp no)
 		(fields_autoplaced yes)
-		(property "Reference" "#PWR0113"
+		(property "Reference" "#PWR0110"
 			(at 80.01 101.6 0)
 			(hide yes)
@@
 			(project "arcticvideo"
 				(path "/9e9873e7-449f-4340-a6d8-702e1fa8c41f/c3f70c33-0f2d-4a7e-8d0b-73a0e9183494"
-					(reference "#PWR0113")
+					(reference "#PWR0110")
 					(unit 1)
 				)
@@
 			)
 		)
-		(property "Footprint" ""
+		(property "Footprint" "Capacitor_SMD:C_0402_1005Metric"
 			(at 84.1248 83.82 0)
 			(hide yes)
@@
 			)
 		)
-		(property "Footprint" ""
+		(property "Footprint" "Capacitor_SMD:C_0402_1005Metric"
 			(at 73.9648 83.82 0)
 			(hide yes)
@@
 			)
 		)
-		(property "Footprint" ""
+		(property "Footprint" "Capacitor_SMD:C_0402_1005Metric"
 			(at 242.8748 71.12 0)
 			(hide yes)
@@
 		(dnp no)
 		(fields_autoplaced yes)
-		(property "Reference" "#PWR0114"
+		(property "Reference" "#PWR0111"
 			(at 151.13 99.06 0)
 			(hide yes)
@@
 			(project "arcticvideo"
 				(path "/9e9873e7-449f-4340-a6d8-702e1fa8c41f/c3f70c33-0f2d-4a7e-8d0b-73a0e9183494"
-					(reference "#PWR0114")
+					(reference "#PWR0111")
 					(unit 1)
 				)
@@
 		(dnp no)
 		(fields_autoplaced yes)
-		(property "Reference" "#PWR0112"
+		(property "Reference" "#PWR0109"
 			(at 67.31 80.01 0)
 			(hide yes)
@@
 			(project "arcticvideo"
 				(path "/9e9873e7-449f-4340-a6d8-702e1fa8c41f/c3f70c33-0f2d-4a7e-8d0b-73a0e9183494"
-					(reference "#PWR0112")
+					(reference "#PWR0109")
 					(unit 1)
 				)
@@
 		(dnp no)
 		(fields_autoplaced yes)
-		(property "Reference" "#PWR0115"
+		(property "Reference" "#PWR0112"
 			(at 194.31 76.2 0)
 			(hide yes)
@@
 			(project "arcticvideo"
 				(path "/9e9873e7-449f-4340-a6d8-702e1fa8c41f/c3f70c33-0f2d-4a7e-8d0b-73a0e9183494"
-					(reference "#PWR0115")
+					(reference "#PWR0112")
 					(unit 1)
 				)
@@
 		(dnp no)
 		(fields_autoplaced yes)
-		(property "Reference" "#PWR0116"
+		(property "Reference" "#PWR0113"
 			(at 194.31 95.25 0)
 			(hide yes)
@@
 			(project "arcticvideo"
 				(path "/9e9873e7-449f-4340-a6d8-702e1fa8c41f/c3f70c33-0f2d-4a7e-8d0b-73a0e9183494"
-					(reference "#PWR0116")
+					(reference "#PWR0113")
 					(unit 1)
 				)
@@
 			)
 		)
-		(property "Footprint" "SG-210STF_EPS"
+		(property "Footprint" "arcticvideo:SG-210STF_EPS"
 			(at 217.678 90.17 0)
 			(hide yes)
@@
 		(dnp no)
 		(fields_autoplaced yes)
-		(property "Reference" "#PWR0118"
+		(property "Reference" "#PWR0115"
 			(at 252.73 78.74 0)
 			(hide yes)
@@
 			(project "arcticvideo"
 				(path "/9e9873e7-449f-4340-a6d8-702e1fa8c41f/c3f70c33-0f2d-4a7e-8d0b-73a0e9183494"
-					(reference "#PWR0118")
-					(unit 1)
-				)
+					(reference "#PWR0115")
+					(unit 1)
+				)
