File: hardware/clock.kicad_sch (KiCad schematic)
At the start: 6 parts

Commit message: finished pcb
Parts:
- renumbered R47 to R48
Changed lines of the file:
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@@
 		(dnp no)
 		(fields_autoplaced yes)
-		(property "Reference" "R47"
+		(property "Reference" "R48"
 			(at 123.19 86.3599 0)
 			(show_name no)
@@
 			(project "arcticvideo"
 				(path "/9e9873e7-449f-4340-a6d8-702e1fa8c41f/c3f70c33-0f2d-4a7e-8d0b-73a0e9183494"
-					(reference "R47")
+					(reference "R48")
 					(unit 1)
 				)
@@
 		(dnp no)
 		(fields_autoplaced yes)
-		(property "Reference" "#PWR0114"
+		(property "Reference" "#PWR0116"
 			(at 237.49 71.12 0)
 			(hide yes)
@@
 			(project "arcticvideo"
 				(path "/9e9873e7-449f-4340-a6d8-702e1fa8c41f/c3f70c33-0f2d-4a7e-8d0b-73a0e9183494"
-					(reference "#PWR0114")
+					(reference "#PWR0116")
 					(unit 1)
 				)
@@
 		(dnp no)
 		(fields_autoplaced yes)
-		(property "Reference" "#PWR0110"
+		(property "Reference" "#PWR0112"
 			(at 80.01 101.6 0)
 			(hide yes)
@@
 			(project "arcticvideo"
 				(path "/9e9873e7-449f-4340-a6d8-702e1fa8c41f/c3f70c33-0f2d-4a7e-8d0b-73a0e9183494"
-					(reference "#PWR0110")
+					(reference "#PWR0112")
 					(unit 1)
 				)
@@
 		(dnp no)
 		(fields_autoplaced yes)
-		(property "Reference" "#PWR0111"
+		(property "Reference" "#PWR0113"
 			(at 151.13 99.06 0)
 			(hide yes)
@@
 			(project "arcticvideo"
 				(path "/9e9873e7-449f-4340-a6d8-702e1fa8c41f/c3f70c33-0f2d-4a7e-8d0b-73a0e9183494"
-					(reference "#PWR0111")
+					(reference "#PWR0113")
 					(unit 1)
 				)
@@
 		(dnp no)
 		(fields_autoplaced yes)
-		(property "Reference" "#PWR0109"
+		(property "Reference" "#PWR0111"
 			(at 67.31 80.01 0)
 			(hide yes)
@@
 			(project "arcticvideo"
 				(path "/9e9873e7-449f-4340-a6d8-702e1fa8c41f/c3f70c33-0f2d-4a7e-8d0b-73a0e9183494"
-					(reference "#PWR0109")
+					(reference "#PWR0111")
 					(unit 1)
 				)
@@
 		(dnp no)
 		(fields_autoplaced yes)
-		(property "Reference" "#PWR0112"
+		(property "Reference" "#PWR0114"
 			(at 194.31 76.2 0)
 			(hide yes)
@@
 			(project "arcticvideo"
 				(path "/9e9873e7-449f-4340-a6d8-702e1fa8c41f/c3f70c33-0f2d-4a7e-8d0b-73a0e9183494"
-					(reference "#PWR0112")
+					(reference "#PWR0114")
 					(unit 1)
 				)
@@
 		(dnp no)
 		(fields_autoplaced yes)
-		(property "Reference" "#PWR0113"
+		(property "Reference" "#PWR0115"
 			(at 194.31 95.25 0)
 			(hide yes)
@@
 			(project "arcticvideo"
 				(path "/9e9873e7-449f-4340-a6d8-702e1fa8c41f/c3f70c33-0f2d-4a7e-8d0b-73a0e9183494"
-					(reference "#PWR0113")
+					(reference "#PWR0115")
 					(unit 1)
 				)
@@
 		(dnp no)
 		(fields_autoplaced yes)
-		(property "Reference" "#PWR0115"
+		(property "Reference" "#PWR0117"
 			(at 252.73 78.74 0)
 			(hide yes)
@@
 			(project "arcticvideo"
 				(path "/9e9873e7-449f-4340-a6d8-702e1fa8c41f/c3f70c33-0f2d-4a7e-8d0b-73a0e9183494"
-					(reference "#PWR0115")
-					(unit 1)
-				)
+					(reference "#PWR0117")
+					(unit 1)
+				)

Commit message: added changed
Parts:
- C131: Arrow Price/Stock (none) -> $0.5280
- C132, C133: Arrow Price/Stock (none) -> $1.0332
- R48: Arrow Price/Stock (none) -> $0.5240
- XTAL1: Arrow Price/Stock (none) -> $2.6764
- XTAL2: Arrow Price/Stock (none) -> $1.4362
Changed lines of the file:
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@@
+			)
+		)
+		(property "Arrow Price/Stock" "$0.5240"
+			(at 120.65 87.63 0)
+			(hide yes)
+			(show_name no)
+			(do_not_autoplace no)
+			(effects
+				(font
+					(size 1.27 1.27)
+				)
 			)
 		)
@@
 			)
 		)
+		(property "Arrow Price/Stock" "$2.6764"
+			(at 97.79 78.74 0)
+			(hide yes)
+			(show_name no)
+			(do_not_autoplace no)
+			(effects
+				(font
+					(size 1.27 1.27)
+				)
+			)
+		)
 		(pin "4"
 		)
@@
 			)
 		)
+		(property "Arrow Price/Stock" "$1.0332"
+			(at 85.09 87.63 90)
+			(hide yes)
+			(show_name no)
+			(do_not_autoplace no)
+			(effects
+				(font
+					(size 1.27 1.27)
+				)
+			)
+		)
 		(pin "1"
 		)
@@
 			)
 		)
+		(property "Arrow Price/Stock" "$0.5280"
+			(at 74.93 87.63 90)
+			(hide yes)
+			(show_name no)
+			(do_not_autoplace no)
+			(effects
+				(font
+					(size 1.27 1.27)
+				)
+			)
+		)
 		(pin "1"
 		)
@@
 		(property "Description" "Unpolarized capacitor"
 			(at 243.84 74.93 0)
+			(hide yes)
+			(show_name no)
+			(do_not_autoplace no)
+			(effects
+				(font
+					(size 1.27 1.27)
+				)
+			)
+		)
+		(property "Arrow Price/Stock" "$1.0332"
+			(at 243.84 74.93 90)
 			(hide yes)
 			(show_name no)
@@
 			(at 198.12 78.74 0)
 			(hide yes)
+			(show_name no)
+			(do_not_autoplace no)
+			(effects
+				(font
+					(size 1.27 1.27)
+				)
+			)
+		)
+		(property "Arrow Price/Stock" "$1.4362"
+			(at 198.12 78.74 0)
+			(hide yes)
