File: hardware/pcie.kicad_sch (KiCad schematic)
At the start: 12 parts, among them J2 Bus_PCI_Express_x4, U8 XC7A35T-2FGG484C, U9 PESD5V0L2BT

Commit message: last commit for a while, i have to change the fpga and i dont have the time, money, or motivation to do that
Parts:
- added C102, C95, C98, C99: 0.1u, symbol Device:C
- added C106, C107: 22u, symbol Device:C
- added C89: 2.2u, symbol Device:C
- added C90: 10u, symbol Device:C
- added C91, C92, C94: 4.7u, symbol Device:C
- added L3: 10u, symbol Device:L
- added R17, R20: 100k, symbol Device:R
- added R18: 1k, symbol Device:R
- added R19: 24.9k, symbol Device:R
- added R21, R?: 12.1k, symbol Device:R
- added U10: TPS62175DQCR, DQC0010A, symbol arcticvideo:TPS62175DQCR
- added U11: AMS1117-ADJ, SOT_AMS1117-2.5_AMS, symbol arcticvideo:AMS1117-ADJ
- added U?: XC7A75T-2FGG484C, FGG484ARTIX-7_AMD, symbol arcticvideo:XC7A75T-2FGG484C
- renumbered C5 to C100, C4 to C101, C3 to C103, C2 to C104, C1 to C105, C8 to C93, C7 to C96, C6 to C97, J2 to J4, R1 to R22, U8 to U1, U9 to U12
Connections:
- net +12V: now also C89.2, U10.2 (VIN), U10.3 (EN), U10.8 (SLEEP)
- net +3V3: now also C90.2, U11.3 (INPUT)
- net GND: now also C102.1, C106.1, C107.1, C89.1, C90.1, C91.1, C92.1, C94.1, C95.1, C98.1, C99.1, R18.2, R20.1, R21.2, R?.2, U10.1 (PGND), U10.11 (PAD), U10.4 (NC), U10.6 (AGND), U11.1 (ADJ/GND)
- net PERn0: now also U?.A8 (MGTPRXN0_216)
- net PERn1: now also U?.C11 (MGTPRXN1_216)
- net PERn2: now also U?.A10 (MGTPRXN2_216)
- net PERn3: now also U?.C9 (MGTPRXN3_216)
- net PERp0: now also U?.B8 (MGTPRXP0_216)
- net PERp1: now also U?.D11 (MGTPRXP1_216)
- net PERp2: now also U?.B10 (MGTPRXP2_216)
- net PERp3: now also U?.D9 (MGTPRXP3_216)
- net PETn0: now also U?.A4 (MGTPTXN0_216)
- net PETn1: now also U?.C5 (MGTPTXN1_216)
- net PETn2: now also U?.A6 (MGTPTXN2_216)
- net PETn3: now also U?.C7 (MGTPTXN3_216)
- net PETp0: now also U?.B4 (MGTPTXP0_216)
- net PETp1: now also U?.D5 (MGTPTXP1_216)
- net PETp2: now also U?.B6 (MGTPTXP2_216)
- net PETp3: now also U?.D7 (MGTPTXP3_216)
- net PRESET: now also U?.P20 (IO_0_14)
- net REFCLKN: now also U?.E6 (MGTREFCLK0N_216)
- net REFCLKP: now also U?.F6 (MGTREFCLK0P_216)
- net +1V25: now reaches U1.B11 (MGTAVTT)
- net +1V25: now also U1.B5 (MGTAVTT), U1.B7 (MGTAVTT), U1.B9 (MGTAVTT), U1.C4 (MGTAVTT), U1.C8 (MGTAVTT), C102.2, C107.2, C91.2, C94.2, C98.2, R18.1, U11.2 (OUTPUT)
- net MGT+1V0: now reaches U1.D10 (MGTAVCC)
- net MGT+1V0: now also U1.D6 (MGTAVCC), U1.E8 (MGTAVCC), U1.F7 (MGTAVCC), U1.F9 (MGTAVCC), C106.2, C92.2, C95.2, C99.2, L3.2, R17.2, R19.2, U10.10 (VOS)
- net at U1.F8 (MGTRREF_216): now also R21.1
- net CCLK_0: now reaches U1.L12 (CCLK_0)
- net CCLK_0: now also U?.L12 (CCLK_0)
- new net: R19.1, R20.2, U10.5 (FB)
- new net: R?.1, U?.F8 (MGTRREF_216)
- new net: L3.1, U10.9 (SW)
- new net: R17.1, U10.7 (PG)
- no-connect marks 0 -> 3
Other:
- moved on the sheet: U1A

Commit message: finished schematic!!! :D (before peer review)
Parts:
- removed R21, R?: 12.1k, symbol Device:R
- removed U1: XC7A35T-2FGG484C, FGG484_AMD, symbol arcticvideo:XC7A35T-2FGG484C
- removed U?: XC7A75T-2FGG484C, FGG484ARTIX-7_AMD, symbol arcticvideo:XC7A75T-2FGG484C
- added R37, R38, R39: 10k, symbol Device:R
Connections:
- net +3V3: now also R37.2, R38.2, R39.2
- net GND: now also J4.A12 (GND), J4.A15 (GND), J4.A18 (GND), J4.A20 (GND), J4.A23 (GND), J4.A24 (GND), J4.A27 (GND), J4.A28 (GND), J4.A31 (GND), J4.A4 (GND), J4.B13 (GND), J4.B16 (GND), J4.B18 (GND), J4.B21 (GND), J4.B22 (GND), J4.B25 (GND), J4.B26 (GND), J4.B29 (GND), J4.B32 (GND), J4.B4 (GND), J4.B7 (GND)
- net at J4.B11 (~{WAKE}): now also R37.1
- net at J4.B5 (SMCLK): now also R38.1
- net at J4.B6 (SMDAT): now also R39.1
- net PRESET renamed PERST
- no-connect marks 3 -> 12
Other:
- note removed: "can move to any io pin based on need :3"
- moved on the sheet: C100, C101, C102, C103, C104, C105, C106, C107, C89, C90, C91, C92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

Commit message: readable changes
Parts:
- removed C107: 22u, symbol Device:C
- removed R18: 1k, symbol Device:R
- added C130: 22u, symbol Device:C
- added R48: 1k, symbol Device:R
- renumbered C89 to C112, C93 to C113, C96 to C114, C97 to C115, C100 to C116, C101 to C117, C103 to C118, C104 to C119, C105 to C120, C106 to C121, C90 to C122, C91 to C123, C92 to C124, C94 to C125, C95 to C126, C98 to C127, C99 to C128, C102 to C129, J4 to J5, R39 to R41, R38 to R42, R17 to R43, R19 to R44, R20 to R45, R37 to R46, R22 to R47, U10 to U11, U11 to U13
Connections:
- net +1V25: now also C130.1, R48.2
- net GND: now also C130.2, R48.1

Commit message: pcb routing
Parts:
- C112, C113, C114, C115, C116, C117, C118, C119, C120, C121, C122, C123, C124, C125, C126, C127, C128, C129, C130: footprint (none) -> Capacitor_SMD:C_0402_1005Metric
- L3: footprint (none) -> Inductor_SMD:L_0402_1005Metric
- R39: renamed from R41; footprint (none) -> Resistor_SMD:R_0402_1005Metric
- R40: renamed from R42; footprint (none) -> Resistor_SMD:R_0402_1005Metric
- R41: renamed from R43; footprint (none) -> Resistor_SMD:R_0402_1005Metric
- R42: renamed from R44; footprint (none) -> Resistor_SMD:R_0402_1005Metric
- R43: renamed from R45; footprint (none) -> Resistor_SMD:R_0402_1005Metric
- R44: renamed from R46; footprint (none) -> Resistor_SMD:R_0402_1005Metric
- R45: renamed from R47; footprint (none) -> Resistor_SMD:R_0402_1005Metric
- R46: renamed from R48; footprint (none) -> Resistor_SMD:R_0402_1005Metric
- U11: footprint DQC0010A -> arcticvideo:DQC0010A
- U12: footprint SOT23_NEX -> arcticvideo:SOT23_NEX
- U13: footprint SOT_AMS1117-2.5_AMS -> arcticvideo:SOT_AMS1117-2.5_AMS
