File: hardware/pcie.kicad_sch (KiCad schematic)
At the start: 32 parts, among them J5 Bus_PCI_Express_x4, U11 TPS62175DQCR, U12 PESD5V0L2BT, U13 AMS1117-ADJ

Commit message: finished pcb
Parts:
- renumbered R39 to R40, R40 to R41, R41 to R42, R42 to R43, R43 to R44, R44 to R45, R45 to R46, R46 to R47
Changed lines of the file:
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@@
 		(dnp no)
 		(fields_autoplaced yes)
-		(property "Reference" "#PWR092"
+		(property "Reference" "#PWR094"
 			(at 53.34 85.09 0)
 			(hide yes)
@@
 			(project "arcticvideo"
 				(path "/9e9873e7-449f-4340-a6d8-702e1fa8c41f/7a2273a0-83e2-422b-8543-03665cb9eb61"
-					(reference "#PWR092")
+					(reference "#PWR094")
 					(unit 1)
 				)
@@
 		(dnp no)
 		(fields_autoplaced yes)
-		(property "Reference" "R43"
+		(property "Reference" "R44"
 			(at 107.95 66.0401 0)
 			(show_name no)
@@
 			(project "arcticvideo"
 				(path "/9e9873e7-449f-4340-a6d8-702e1fa8c41f/7a2273a0-83e2-422b-8543-03665cb9eb61"
-					(reference "R43")
+					(reference "R44")
 					(unit 1)
 				)
@@
 		(dnp no)
 		(fields_autoplaced yes)
-		(property "Reference" "#PWR0100"
+		(property "Reference" "#PWR0102"
 			(at 152.4 58.42 0)
 			(hide yes)
@@
 			(project "arcticvideo"
 				(path "/9e9873e7-449f-4340-a6d8-702e1fa8c41f/7a2273a0-83e2-422b-8543-03665cb9eb61"
-					(reference "#PWR0100")
+					(reference "#PWR0102")
 					(unit 1)
 				)
@@
 		(dnp no)
 		(fields_autoplaced yes)
-		(property "Reference" "#PWR0105"
+		(property "Reference" "#PWR0107"
 			(at 210.82 135.89 0)
 			(hide yes)
@@
 			(project "arcticvideo"
 				(path "/9e9873e7-449f-4340-a6d8-702e1fa8c41f/7a2273a0-83e2-422b-8543-03665cb9eb61"
-					(reference "#PWR0105")
+					(reference "#PWR0107")
 					(unit 1)
 				)
@@
 		(dnp no)
 		(fields_autoplaced yes)
-		(property "Reference" "#PWR0106"
+		(property "Reference" "#PWR0108"
 			(at 210.82 151.13 0)
 			(hide yes)
@@
 			(project "arcticvideo"
 				(path "/9e9873e7-449f-4340-a6d8-702e1fa8c41f/7a2273a0-83e2-422b-8543-03665cb9eb61"
-					(reference "#PWR0106")
+					(reference "#PWR0108")
 					(unit 1)
 				)
@@
 		(dnp no)
 		(fields_autoplaced yes)
-		(property "Reference" "R40"
+		(property "Reference" "R41"
 			(at 81.28 121.9201 0)
 			(show_name no)
@@
 			(project "arcticvideo"
 				(path "/9e9873e7-449f-4340-a6d8-702e1fa8c41f/7a2273a0-83e2-422b-8543-03665cb9eb61"
-					(reference "R40")
+					(reference "R41")
 					(unit 1)
 				)
@@
 		(dnp no)
 		(fields_autoplaced yes)
-		(property "Reference" "#PWR098"
+		(property "Reference" "#PWR0100"
 			(at 137.16 165.1 0)
 			(hide yes)
@@
 			(project "arcticvideo"
 				(path "/9e9873e7-449f-4340-a6d8-702e1fa8c41f/7a2273a0-83e2-422b-8543-03665cb9eb61"
-					(reference "#PWR098")
+					(reference "#PWR0100")
 					(unit 1)
 				)
@@
 		(dnp no)
 		(fields_autoplaced yes)
-		(property "Reference" "#PWR099"
+		(property "Reference" "#PWR0101"
 			(at 140.97 123.19 0)
 			(hide yes)
@@
 			(project "arcticvideo"
 				(path "/9e9873e7-449f-4340-a6d8-702e1fa8c41f/7a2273a0-83e2-422b-8543-03665cb9eb61"
-					(reference "#PWR099")
+					(reference "#PWR0101")
 					(unit 1)
 				)
@@
 		(dnp no)
 		(fields_autoplaced yes)
-		(property "Reference" "#PWR091"
+		(property "Reference" "#PWR093"
 			(at 34.29 62.23 0)
 			(hide yes)
@@
 			(project "arcticvideo"
 				(path "/9e9873e7-449f-4340-a6d8-702e1fa8c41f/7a2273a0-83e2-422b-8543-03665cb9eb61"
-					(reference "#PWR091")
+					(reference "#PWR093")
 					(unit 1)
 				)
@@
 		(dnp no)
 		(fields_autoplaced yes)
-		(property "Reference" "#PWR0107"
+		(property "Reference" "#PWR0109"
 			(at 224.79 48.26 0)
 			(hide yes)
@@
 			(project "arcticvideo"
 				(path "/9e9873e7-449f-4340-a6d8-702e1fa8c41f/7a2273a0-83e2-422b-8543-03665cb9eb61"
-					(reference "#PWR0107")
+					(reference "#PWR0109")
 					(unit 1)
 				)
@@
 		(dnp no)
 		(fields_autoplaced yes)
-		(property "Reference" "#PWR096"
+		(property "Reference" "#PWR098"
 			(at 101.6 191.77 0)
 			(hide yes)
@@
 			(project "arcticvideo"
 				(path "/9e9873e7-449f-4340-a6d8-702e1fa8c41f/7a2273a0-83e2-422b-8543-03665cb9eb61"
-					(reference "#PWR096")
+					(reference "#PWR098")
 					(unit 1)
 				)
@@
 		(dnp no)
 		(fields_autoplaced yes)
-		(property "Reference" "R46"
+		(property "Reference" "R47"
 			(at 236.22 53.3399 0)
 			(show_name no)
@@
 			(project "arcticvideo"
 				(path "/9e9873e7-449f-4340-a6d8-702e1fa8c41f/7a2273a0-83e2-422b-8543-03665cb9eb61"
-					(reference "R46")
+					(reference "R47")
 					(unit 1)
 				)
@@
 		(dnp no)
 		(fields_autoplaced yes)
-		(property "Reference" "#PWR0101"
+		(property "Reference" "#PWR0103"
 			(at 153.67 167.64 0)
 			(hide yes)
@@
 			(project "arcticvideo"
 				(path "/9e9873e7-449f-4340-a6d8-702e1fa8c41f/7a2273a0-83e2-422b-8543-03665cb9eb61"
-					(reference "#PWR0101")
+					(reference "#PWR0103")
 					(unit 1)
 				)
@@
 		(dnp no)
 		(fields_autoplaced yes)
-		(property "Reference" "R44"
+		(property "Reference" "R45"
 			(at 138.43 127.0001 0)
 			(show_name no)
@@
 			(project "arcticvideo"
 				(path "/9e9873e7-449f-4340-a6d8-702e1fa8c41f/7a2273a0-83e2-422b-8543-03665cb9eb61"
-					(reference "R44")
+					(reference "R45")
 					(unit 1)
 				)
@@
 		(dnp no)
 		(fields_autoplaced yes)
-		(property "Reference" "#PWR0103"
+		(property "Reference" "#PWR0105"
 			(at 210.82 109.22 0)
 			(hide yes)
@@
 			(project "arcticvideo"
 				(path "/9e9873e7-449f-4340-a6d8-702e1fa8c41f/7a2273a0-83e2-422b-8543-03665cb9eb61"
-					(reference "#PWR0103")
+					(reference "#PWR0105")
 					(unit 1)
 				)
@@
 		(dnp no)
 		(fields_autoplaced yes)
-		(property "Reference" "#PWR093"
+		(property "Reference" "#PWR095"
 			(at 78.74 115.57 0)
 			(hide yes)
@@
 			(project "arcticvideo"
 				(path "/9e9873e7-449f-4340-a6d8-702e1fa8c41f/7a2273a0-83e2-422b-8543-03665cb9eb61"
-					(reference "#PWR093")
+					(reference "#PWR095")
 					(unit 1)
 				)
@@
 		(dnp no)
 		(fields_autoplaced yes)
-		(property "Reference" "#PWR094"
+		(property "Reference" "#PWR096"
 			(at 93.98 86.36 0)
 			(hide yes)
@@
 			(project "arcticvideo"
 				(path "/9e9873e7-449f-4340-a6d8-702e1fa8c41f/7a2273a0-83e2-422b-8543-03665cb9eb61"
-					(reference "#PWR094")
+					(reference "#PWR096")
 					(unit 1)
 				)
@@
 		(dnp no)
 		(fields_autoplaced yes)
-		(property "Reference" "#PWR090"
+		(property "Reference" "#PWR092"
 			(at 31.75 44.45 0)
 			(hide yes)
@@
 			(project "arcticvideo"
 				(path "/9e9873e7-449f-4340-a6d8-702e1fa8c41f/7a2273a0-83e2-422b-8543-03665cb9eb61"
-					(reference "#PWR090")
+					(reference "#PWR092")
 					(unit 1)
 				)
@@
 		(dnp no)
 		(fields_autoplaced yes)
-		(property "Reference" "R41"
+		(property "Reference" "R42"
 			(at 96.52 55.8801 0)
 			(show_name no)
@@
 			(project "arcticvideo"
 				(path "/9e9873e7-449f-4340-a6d8-702e1fa8c41f/7a2273a0-83e2-422b-8543-03665cb9eb61"
-					(reference "R41")
+					(reference "R42")
 					(unit 1)
 				)
@@
 		(dnp no)
 		(fields_autoplaced yes)
-		(property "Reference" "#PWR095"
+		(property "Reference" "#PWR097"
 			(at 99.06 113.03 0)
 			(hide yes)
@@
 			(project "arcticvideo"
 				(path "/9e9873e7-449f-4340-a6d8-702e1fa8c41f/7a2273a0-83e2-422b-8543-03665cb9eb61"
-					(reference "#PWR095")
+					(reference "#PWR097")
 					(unit 1)
 				)
@@
 		(dnp no)
 		(fields_autoplaced yes)
-		(property "Reference" "R39"
+		(property "Reference" "R40"
 			(at 72.39 124.4601 0)
 			(show_name no)
@@
 			(project "arcticvideo"
 				(path "/9e9873e7-449f-4340-a6d8-702e1fa8c41f/7a2273a0-83e2-422b-8543-03665cb9eb61"
-					(reference "R39")
+					(reference "R40")
 					(unit 1)
 				)
@@
 		(dnp no)
 		(fields_autoplaced yes)
-		(property "Reference" "R42"
+		(property "Reference" "R43"
 			(at 107.95 58.4201 0)
 			(show_name no)
@@
 			(project "arcticvideo"
 				(path "/9e9873e7-449f-4340-a6d8-702e1fa8c41f/7a2273a0-83e2-422b-8543-03665cb9eb61"
-					(reference "R42")
+					(reference "R43")
 					(unit 1)
 				)
@@
 		(dnp no)
 		(fields_autoplaced yes)
-		(property "Reference" "#PWR097"
+		(property "Reference" "#PWR099"
 			(at 121.92 46.99 0)
 			(hide yes)
@@
 			(project "arcticvideo"
 				(path "/9e9873e7-449f-4340-a6d8-702e1fa8c41f/7a2273a0-83e2-422b-8543-03665cb9eb61"
-					(reference "#PWR097")
+					(reference "#PWR099")
 					(unit 1)
 				)
@@
 		(dnp no)
 		(fields_autoplaced yes)
-		(property "Reference" "#PWR0102"
+		(property "Reference" "#PWR0104"
 			(at 160.02 73.66 0)
 			(hide yes)
@@
 			(project "arcticvideo"
 				(path "/9e9873e7-449f-4340-a6d8-702e1fa8c41f/7a2273a0-83e2-422b-8543-03665cb9eb61"
-					(reference "#PWR0102")
+					(reference "#PWR0104")
 					(unit 1)
 				)
@@
 		(dnp no)
 		(fields_autoplaced yes)
-		(property "Reference" "#PWR0104"
+		(property "Reference" "#PWR0106"
 			(at 210.82 124.46 0)
 			(hide yes)
@@
 			(project "arcticvideo"
 				(path "/9e9873e7-449f-4340-a6d8-702e1fa8c41f/7a2273a0-83e2-422b-8543-03665cb9eb61"
-					(reference "#PWR0104")
+					(reference "#PWR0106")
 					(unit 1)
 				)
@@
 		(dnp no)
 		(fields_autoplaced yes)
-		(property "Reference" "#PWR0108"
+		(property "Reference" "#PWR0110"
 			(at 254 54.61 0)
 			(hide yes)
@@
 			(project "arcticvideo"
 				(path "/9e9873e7-449f-4340-a6d8-702e1fa8c41f/7a2273a0-83e2-422b-8543-03665cb9eb61"
-					(reference "#PWR0108")
+					(reference "#PWR0110")
 					(unit 1)
 				)
@@
 		(dnp no)
 		(fields_autoplaced yes)
-		(property "Reference" "R45"
+		(property "Reference" "R46"
 			(at 146.05 162.5601 0)
 			(show_name no)
@@
 			(project "arcticvideo"
 				(path "/9e9873e7-449f-4340-a6d8-702e1fa8c41f/7a2273a0-83e2-422b-8543-03665cb9eb61"
-					(reference "R45")
+					(reference "R46")
 					(unit 1)
 				)

Commit message: added changed
Parts:
- C112, C121, C130: Arrow Price/Stock (none) -> $0.2580
- C113, C114, C115, C116, C117, C118, C119, C120: Arrow Price/Stock (none) -> $0.2520
- C122, L3: Arrow Price/Stock (none) -> $1.9152
- C123, C124, C125: Arrow Price/Stock (none) -> $3.2704
- C126, C127, C128, C129: Arrow Price/Stock (none) -> $1.0332
- J5: now left out of the parts list
- R40, R41, R45, R46: Arrow Price/Stock (none) -> $0.2552
- R42, R44: Arrow Price/Stock (none) -> $0.0640
- R43: Arrow Price/Stock (none) -> $0.0280
- R47: Arrow Price/Stock (none) -> $0.1000
- U11: Arrow Price/Stock (none) -> $2.6122
- U12: Arrow Price/Stock (none) -> $0.3306
- U13: Arrow Price/Stock (none) -> $1.3188
