File: hardware/power.kicad_sch (KiCad schematic)
At the start: 5 parts, among them U1 XC7A35T-2FGG484C, U4 AMS1117-1.8, U5 AMS1117-ADJ, U6 MP2307DN-LF-Z, U7 MP2307DN-LF-Z

Commit message: last commit for a while, i have to change the fpga and i dont have the time, money, or motivation to do that
Parts:
- removed U7: MP2307DN-LF-Z, IC8_MP2307_MNP, symbol arcticvideo:MP2307DN-LF-Z
- added C1: 100u, symbol Device:C
- added C10, C11, C13, C18, C20, C25, C26, C29, C48, C49, C50, C51, C52, C53, C54, C55, C56, C57, C58, C59, C60, C61, C62, C63, C64, C65, C66, C67, C68, C69, C70, C71, C8, C?: 0.47u, symbol Device:C
- added C12, C19, C2, C30, C31, C32, C33, C34, C35, C?: 47u, symbol Device:C
- added C14, C15, C36, C37, C38, C39, C40, C41, C42, C43, C44, C45, C46, C47, C7, C9: 4.7u, symbol Device:C
- added C16, C17: 10n, symbol Device:C
- added C21, C22: 3.9n, symbol Device:C
- added C23, C24, C27, C28: 22u, symbol Device:C
- added C3, C4, C5, C6: 10u, symbol Device:C
- added C72, C?: 0.1u, symbol Device:C
- added L1, L2: 10u, symbol Device:L
- added R1, R2: 100k, symbol Device:R
- added R10: 800, symbol Device:R
- added R3: 2.2k, symbol Device:R
- added R4: 180, symbol Device:R
- added R5, R6: 6.8k, symbol Device:R
- added R7, R8: 10k, symbol Device:R
- added R9: 26.1k, symbol Device:R
- added U3: MP2307DN-LF-Z, IC8_MP2307_MNP, symbol arcticvideo:MP2307DN-LF-Z
- added U? (x3): XC7A75T-2FGG484C, FGG484ARTIX-7_AMD, symbol arcticvideo:XC7A75T-2FGG484C
- renumbered U6 to U2, U5 to U4, U4 to U5
Connections:
- net GND: now also U1.K9 (GNDADC_0), U1.L9 (VREFN_0), U2.4 (GND), U2.8 (SS), U2.EPAD, U5.1 (GROUND/ADJUST), C1.1, C10.1, C11.1, C12.1, C13.1, C14.1, C15.1, C18.1, C19.1, C2.1, C20.1, C23.1, C24.1, C25.1, C26.1, C27.2, C28.2, C29.1, C3.1, C30.1, C31.1, C32.1, C33.1, C34.1, C35.1, C36.1, C37.1, C38.1, C39.1, C4.1, C40.1, C41.1, C42.1, C43.1, C44.1, C45.1, C46.1, C47.1, C48.1, C49.1, C5.1, C50.1, C51.1, C52.1, C53.1, C54.1, C55.1, C56.1, C57.1, C58.1, C59.1, C6.1, C60.1, C61.1, C62.1, C63.1, C64.1, C65.1, C66.1, C67.1, C68.1, C69.1, C7.1, C70.1, C71.1, C72.1, C8.1, C9.1, C?.1, C?.1, C?.1, R4.2, R5.1, R6.1, R7.2, R8.2, U3.4 (GND), U3.8 (SS), U3.EPAD, U?.A11 (GND), U?.A12 (GND), U?.A2 (GND), U?.A22 (GND), U?.A3 (GND), U?.A5 (GND), U?.A7 (GND), U?.A9 (GND), U?.AA12 (GND), U?.AA2 (GND), U?.AA22 (GND), U?.AB19 (GND), U?.AB9 (GND), U?.B12 (GND), U?.B19 (GND), U?.B3 (GND), U?.C10 (GND), U?.C12 (GND), U?.C16 (GND), U?.C3 (GND), U?.C6 (GND), U?.D12 (GND), U?.D13 (GND), U?.D3 (GND), U?.D4 (GND), U?.D8 (GND), U?.E11 (GND), U?.E20 (GND), U?.E4 (GND), U?.E5 (GND), U?.E7 (GND), U?.E9 (GND), U?.F11 (GND), U?.F17 (GND), U?.F5 (GND), U?.G10 (GND), U?.G12 (GND), U?.G14 (GND), U?.G5 (GND), U?.G6 (GND), U?.G7 (GND), U?.G8 (GND), U?.G9 (GND), U?.H1 (GND), U?.H11 (GND), U?.H21 (GND), U?.H7 (GND), U?.H9 (GND), U?.J10 (GND), U?.J12 (GND), U?.J18 (GND), U?.J8 (GND), U?.K11 (GND), U?.K15 (GND), U?.K5 (GND), U?.K7 (GND), U?.K9 (GNDADC_0), U?.L2 (GND), U?.L22 (GND), U?.L8 (GND), U?.L9 (VREFN_0), U?.M11 (GND), U?.M19 (GND), U?.M7 (GND), U?.N16 (GND), U?.N6 (GND), U?.N8 (GND), U?.P11 (GND), U?.P13 (GND), U?.P3 (GND), U?.P7 (GND), U?.P9 (GND), U?.R10 (GND), U?.R12 (GND), U?.R20 (GND), U?.R8 (GND), U?.T11 (GND), U?.T17 (GND), U?.T7 (GND), U?.T9 (GND), U?.U14 (GND), U?.U4 (GND), U?.V1 (GND), U?.V11 (GND), U?.V21 (GND), U?.W18 (GND), U?.W8 (GND), U?.Y15 (GND), U?.Y5 (GND)
- net at U4.1 (ADJ/GND): now also R3.2, R4.1
- net +1V35: now reaches U4.2 (OUTPUT)
- net +1V35: now also U1.AA7 (VCCO_34), U1.AB4 (VCCO_34), U1.C1 (VCCO_35), U1.F2 (VCCO_35), U1.H6 (VCCO_35), U1.J3 (VCCO_35), U1.M4 (VCCO_35), U1.N1 (VCCO_35), U1.R5 (VCCO_34), U1.T2 (VCCO_34), U1.V6 (VCCO_34), U1.W3 (VCCO_34), C23.2, C34.2, C35.2, C40.2, C41.2, C46.2, C47.2, C52.2, C53.2, C58.2, C59.2, C64.2, C65.2, C70.2, C71.2, R3.1, U?.AA7 (VCCO_34), U?.AB4 (VCCO_34), U?.C1 (VCCO_35), U?.F2 (VCCO_35), U?.H6 (VCCO_35), U?.J3 (VCCO_35), U?.M4 (VCCO_35), U?.N1 (VCCO_35), U?.R5 (VCCO_34), U?.T2 (VCCO_34), U?.V6 (VCCO_34), U?.W3 (VCCO_34)
- net +3V3: now reaches U4.3 (INPUT)
- net +3V3: now also U1.AA17 (VCCO_13), U1.AB14 (VCCO_13), U1.F12 (VCCO_0), U1.M14 (VCCO_14), U1.P18 (VCCO_14), U1.R15 (VCCO_14), U1.T12 (VCCO_0), U1.T22 (VCCO_14), U1.U19 (VCCO_14), U1.V16 (VCCO_13), U1.W13 (VCCO_13), U1.Y10 (VCCO_13), U1.Y20 (VCCO_14), U5.3 (VIN), C19.2, C27.1, C3.2, C30.2, C31.2, C36.2, C37.2, C4.2, C42.2, C43.2, C48.2, C49.2, C54.2, C55.2, C60.2, C61.2, C66.2, C67.2, L1.2, R9.2, U?.AA17 (VCCO_13), U?.AB14 (VCCO_13), U?.F12 (VCCO_0), U?.M14 (VCCO_14), U?.P18 (VCCO_14), U?.R15 (VCCO_14), U?.T12 (VCCO_0), U?.T22 (VCCO_14), U?.U19 (VCCO_14), U?.V16 (VCCO_13), U?.W13 (VCCO_13), U?.Y10 (VCCO_13), U?.Y20 (VCCO_14)
- net at U2.1 (BS): now also C16.1
- net +12V: now reaches U2.2 (IN)
- net +12V: now also C5.2, C6.2, R1.2, R2.2, U3.2 (IN)
- net at U2.3 (SW): now also C16.2, L1.1
- net at U2.5 (FB): now also R7.1, R9.1
- net at U2.6 (COMP): now also C21.1
- net at U2.7 (EN): now also R1.1
- net +1V0: now reaches U1.H10 (VCCINT)
- net +1V0: now also U1.H8 (VCCINT), U1.J11 (VCCBRAM), U1.J7 (VCCINT), U1.J9 (VCCINT), U1.K8 (VCCINT), U1.L11 (VCCBRAM), U1.L7 (VCCINT), U1.M8 (VCCINT), U1.N11 (VCCBRAM), U1.N7 (VCCINT), U1.P10 (VCCINT), U1.P8 (VCCINT), U1.R7 (VCCINT), U1.R9 (VCCINT), U1.T10 (VCCINT), U1.T8 (VCCINT), C1.2, C10.2, C11.2, C13.2, C2.2, C28.1, C7.2, C8.2, C9.2, C?.2, C?.2, L2.2, R10.2
- net +1V8: now reaches U1.H12 (VCCAUX)
- net +1V8: now also U1.A17 (VCCO_16), U1.B14 (VCCO_16), U1.C21 (VCCO_16), U1.D18 (VCCO_16), U1.E15 (VCCO_16), U1.F22 (VCCO_16), U1.G19 (VCCO_15), U1.H16 (VCCO_15), U1.J13 (VCCO_15), U1.K12 (VCCAUX), U1.K20 (VCCO_15), U1.L17 (VCCO_15), U1.M12 (VCCAUX), U1.N21 (VCCO_15), U1.P12 (VCCAUX), U1.R11 (VCCAUX), U5.2 (VOUT), C12.2, C14.2, C15.2, C18.2, C20.2, C24.2, C25.2, C26.2, C29.2, C32.2, C33.2, C38.2, C39.2, C44.2, C45.2, C50.2, C51.2, C56.2, C57.2, C62.2, C63.2, C68.2, C69.2, U?.A17 (VCCO_16), U?.B14 (VCCO_16), U?.C21 (VCCO_16), U?.D18 (VCCO_16), U?.E15 (VCCO_16), U?.F22 (VCCO_16), U?.G19 (VCCO_15), U?.H16 (VCCO_15), U?.J13 (VCCO_15), U?.K20 (VCCO_15), U?.L17 (VCCO_15), U?.N21 (VCCO_15)
- net at U1.M10 (VREFP_0): now also C72.2
- new net: C?.2, U?.M10 (VREFP_0)
- new net: C17.1, U3.1 (BS)
- new net: C17.2, L2.1, U3.3 (SW)
- new net: R10.1, R8.1, U3.5 (FB)
- new net: R2.1, U3.7 (EN)
- new net: C22.2, R6.2
- new net: C21.2, R5.2
- new net: C22.1, U3.6 (COMP)
- no-connect marks 0 -> 1
Other:
- moved on the sheet: U1F, U1G, U1H, U1I, U2, U4, U5

Commit message: finished schematic!!! :D (before peer review)
Parts:
- removed C72, C?: 0.1u, symbol Device:C
- removed U1: XC7A35T-2FGG484C, FGG484_AMD, symbol arcticvideo:XC7A35T-2FGG484C
- removed U? (x3): XC7A75T-2FGG484C, FGG484ARTIX-7_AMD, symbol arcticvideo:XC7A75T-2FGG484C
- added C? (x8): 0.47u, symbol Device:C
- added C? (x4): 4.7u, symbol Device:C
- added C? (x2): 47u, symbol Device:C
- added R? (x2): 12.1k, symbol Device:R
- added U? (x2): XC7A75T-FGG676, symbol FPGA_Xilinx_Artix7:XC7A75T-FGG676
Connections:
- net +1V0: now also U?.J11 (VCCINT), U?.J13 (VCCINT), U?.K10 (VCCINT), U?.K12 (VCCINT), U?.L11 (VCCINT), U?.L13 (VCCINT), U?.M10 (VCCINT), U?.M12 (VCCADC_0), U?.N13 (VCCBRAM), U?.P10 (VCCINT), U?.R13 (VCCBRAM), U?.T10 (VCCINT), U?.T12 (VCCINT), U?.U11 (VCCINT), U?.U13 (VCCBRAM), U?.V10 (VCCINT), U?.V12 (VCCINT), U?.W13 (VCCBRAM)
- net +1V35: now also C?.2, C?.2, C?.2, C?.2, C?.2, C?.2, C?.2
- net +1V8: now also U?.J9 (VCCAUX), U?.L9 (VCCAUX), U?.N9 (VCCAUX), U?.R9 (VCCAUX), U?.U9 (VCCAUX)
- net +3V3: now also C?.2, C?.2, C?.2, C?.2, C?.2, C?.2, C?.2
- net GND: now also C?.1, C?.1, C?.1, C?.1, C?.1, C?.1, C?.1, C?.1, C?.1, C?.1, C?.1, C?.1, C?.1, C?.1, R?.2, R?.2, U?.A10 (GND), U?.A12 (GND), U?.A14 (GND), U?.A16 (GND), U?.A26 (GND), U?.A6 (GND), U?.A8 (GND), U?.AA14 (GND), U?.AA16 (GND), U?.AA26 (GND), U?.AA6 (GND), U?.AA9 (GND), U?.AB10 (GND), U?.AB12 (GND), U?.AB14 (GND), U?.AB23 (GND), U?.AB3 (GND), U?.AB8 (GND), U?.AB9 (GND), U?.AC15 (GND), U?.AC20 (GND), U?.AC7 (GND), U?.AD11 (GND), U?.AD13 (GND), U?.AD16 (GND), U?.AD6 (GND), U?.AD9 (GND), U?.AE15 (GND), U?.AE24 (GND), U?.AE4 (GND), U?.AE6 (GND), U?.AF1 (GND), U?.AF10 (GND), U?.AF12 (GND), U?.AF14 (GND), U?.AF16 (GND), U?.AF21 (GND), U?.AF6 (GND), U?.AF8 (GND), U?.B15 (GND), U?.B16 (GND), U?.B23 (GND), U?.B3 (GND), U?.B6 (GND), U?.C11 (GND), U?.C13 (GND), U?.C16 (GND), U?.C20 (GND), U?.C6 (GND), U?.C9 (GND), U?.D15 (GND), U?.D17 (GND), U?.D7 (GND), U?.E10 (GND), U?.E12 (GND), U?.E14 (GND), U?.E15 (GND), U?.E24 (GND), U?.E4 (GND), U?.E7 (GND), U?.E8 (GND), U?.E9 (GND), U?.F1 (GND), U?.F14 (GND), U?.F21 (GND), U?.F9 (GND), U?.G10 (GND), U?.G11 (GND), U?.G12 (GND), U?.G13 (GND), U?.G18 (GND), U?.H25 (GND), U?.H5 (GND), U?.J12 (GND), U?.J2 (GND), U?.J22 (GND), U?.K11 (GND), U?.K13 (GND), U?.K19 (GND), U?.K9 (GND), U?.L10 (GND), U?.L12 (GND), U?.L16 (GND), U?.L26 (GND), U?.L6 (GND), U?.M11 (GNDADC_0), U?.M13 (GND), U?.M23 (GND), U?.M3 (GND), U?.M9 (GND), U?.N10 (GND), U?.N20 (GND), U?.P13 (GND), U?.P17 (GND), U?.P7 (GND), U?.P9 (GND), U?.R10 (GND), U?.R24 (GND), U?.R4 (GND), U?.T1 (GND), U?.T11 (GND), U?.T13 (GND), U?.T21 (GND), U?.T9 (GND), U?.U10 (GND), U?.U12 (GND), U?.U18 (GND), U?.U8 (GND), U?.V13 (GND), U?.V15 (GND), U?.V25 (GND), U?.V5 (GND), U?.W12 (GND), U?.W2 (GND), U?.W22 (GND), U?.Y10 (GND), U?.Y11 (GND), U?.Y12 (GND), U?.Y13 (GND), U?.Y19 (GND)
- new net: R?.1, U?.AF15 (MGTRREF_213)
- new net: R?.1, U?.A15 (MGTRREF_216)
- new net MGTAVCC: U?.AA10 (MGTAVCC_G10), U?.AA12 (MGTAVCC_G10), U?.AC11 (MGTAVCC_G10), U?.AC13 (MGTAVCC_G10), U?.AC9 (MGTAVCC_G10), U?.D11 (MGTAVCC_G11), U?.D13 (MGTAVCC_G11), U?.D9 (MGTAVCC_G11), U?.F10 (MGTAVCC_G11), U?.F12 (MGTAVCC_G11)
- new net MGTAVTT: U?.AD15 (MGTAVTT_G10), U?.AD7 (MGTAVTT_G10), U?.AE10 (MGTAVTT_G10), U?.AE12 (MGTAVTT_G10), U?.AE14 (MGTAVTT_G10), U?.AE8 (MGTAVTT_G10), U?.B10 (MGTAVTT_G11), U?.B12 (MGTAVTT_G11), U?.B14 (MGTAVTT_G11), U?.B8 (MGTAVTT_G11), U?.C15 (MGTAVTT_G11), U?.C7 (MGTAVTT_G11)
Other:
- moved on the sheet: C1, C10, C11, C12, C13, C14, C15, C18, C19, C2, C20, C25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

Commit message: readable changes
Parts:
- removed C24: 22u, symbol Device:C
- removed R4: 180, symbol Device:R
- added C25: 22u, symbol Device:C
- added R3: 180, symbol Device:R
- gave numbers to parts that had none: 19
- renumbered C18 to C16, C16 to C17, C17 to C18, C25 to C23, C23 to C24, C29 to C28, C27 to C30, C28 to C31, C30 to C33, C31 to C34, C32 to C35, C33 to C36, C36 to C38, C37 to C39, C38 to C40, C39 to C41, C42 to C43, C43 to C44, C44 to C45, C45 to C46, C54 to C53, C55 to C54, C56 to C55, C57 to C56, C60 to C58, C61 to C59, C62 to C60, C63 to C61, C66 to C63, C67 to C64, C68 to C65, C69 to C66, C34 to C67, C35 to C68, C40 to C70, C41 to C71, C46 to C73, C47 to C74, C52 to C76, C53 to C77, C58 to C79, C59 to C80, C64 to C82, C65 to C83, C70 to C85, C71 to C86, R2 to R1, R1 to R2, R3 to R4
Connections:
- net +1V8: now also C25.1
- net GND: now also C25.2, R3.1
- net at R4.2, U4.1 (ADJ/GND): now also R3.2
- no-connect marks 1 -> 2
Other:
- moved on the sheet: C17, C18, C24, L1, L2, R2, R4

Commit message: pcb routing
Parts:
- removed R11, R12: 12.1k, symbol Device:R
- removed unit 6 of U1
- C1, C10, C11, C12, C13, C14, C15, C16, C17, C18, C19, C2, C20, C21, C22, C23, C24, C25, C26, C27, C28, C29, C3, C30, C31, C32, C33, C34, C35, C36, C37, C38, C39, C4, C40, C41, C42, C43, C44, C45, C46, C47, C48, C49, C5, C50, C51, C52, C53, C54, C55, C56, C57, C58, C59, C6, C60, C61, C62, C63, C64, C65, C66, C67, C68, C69, C7, C70, C71, C72, C73, C74, C75, C76, C77, C78, C79, C8, C80, C81, C82, C83, C84, C85, C86, C87, C9: footprint (none) -> Capacitor_SMD:C_0402_1005Metric
- L1, L2: footprint (none) -> Inductor_SMD:L_0402_1005Metric
- R1, R10, R2, R3, R4, R5, R6, R7, R8, R9: footprint (none) -> Resistor_SMD:R_0402_1005Metric
- U1: footprint (none) -> Package_BGA:Xilinx_FGG676
- U2, U3: footprint IC8_MP2307_MNP -> arcticvideo:IC8_MP2307_MNP
- U4: footprint SOT_AMS1117-2.5_AMS -> arcticvideo:SOT_AMS1117-2.5_AMS
- U5: footprint SOT223_AMS1117-1.8_AMS -> arcticvideo:SOT223_AMS1117-1.8_AMS
