File: hardware/power.kicad_sch (KiCad schematic)
At the start: 104 parts, among them U1 XC7A75T-FGG676, U2 MP2307DN-LF-Z, U3 MP2307DN-LF-Z, U4 AMS1117-ADJ, U5 AMS1117-1.8

Commit message: finished pcb
Parts:
- added H1: MountingHole_Pad, MountingHole:MountingHole_2.7mm_Pad_Via, symbol Mechanical:MountingHole_Pad
- added H2: MountingHole_Pad, MountingHole:MountingHole_3mm_Pad_Via, symbol Mechanical:MountingHole_Pad
- C12, C19, C27, C32, C33, C34, C35, C36, C67, C68, C69: footprint Capacitor_SMD:C_0402_1005Metric -> Capacitor_SMD:C_0603_1608Metric
Connections:
- net GND: now also H1.1, H2.1

Commit message: added changed
Parts:
- C1: Arrow Price/Stock (none) -> $0.4446
- C10, C11, C13, C16, C20, C23, C26, C28, C29, C47, C48, C49, C50, C51, C52, C53, C54, C55, C56, C57, C58, C59, C60, C61, C62, C63, C64, C65, C66, C76, C77, C78, C79, C8, C80, C81, C82, C83, C84, C85, C86, C87: Arrow Price/Stock (none) -> $0.3196
- C12, C19, C2, C27, C32, C33, C34, C35, C36, C67, C68, C69: Arrow Price/Stock (none) -> $5.184
- C14, C15, C37, C38, C39, C40, C41, C42, C43, C44, C45, C46, C7, C70, C71, C72, C73, C74, C75, C9: Arrow Price/Stock (none) -> $3.2704
- C17, C18: Arrow Price/Stock (none) -> $0.0160
- C21, C22: Arrow Price/Stock (none) -> $0.0320
- C24, C25, C30, C31: Arrow Price/Stock (none) -> $0.2580
- C3, C4, C5, C6, L1, L2: Arrow Price/Stock (none) -> $1.9152
- R1, R2: Arrow Price/Stock (none) -> $0.0640
- R10: Arrow Price/Stock (none) -> $0.0820
- R3, R4: Arrow Price/Stock (none) -> $0.0280
- R5, R6: Arrow Price/Stock (none) -> $0.1240
- R7, R8: Arrow Price/Stock (none) -> $0.2552
- R9: Arrow Price/Stock (none) -> $0.0200
- U1: Arrow Price/Stock (none) -> $77.7344
- U2, U3: Arrow Price/Stock (none) -> $14.8452
- U4: Arrow Price/Stock (none) -> $1.3188
- U5: Arrow Price/Stock (none) -> $0.3156
