File: hardware/arcticvideo.kicad_pcb (KiCad board)
At the start: 8 copper layers, 312 x 98.8 mm, 220 parts, among them J1 472720024, J2 Conn_Coaxial, J3 Conn_Coaxial, J5 Bus_PCI_Express_x4, U1 XC7A75T-FGG676, U10 TPS51200DRCR, U11 TPS62175DQCR, U12 PESD5V0L2BT, U13 AMS1117-ADJ, U2 MP2307DN-LF-Z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

Commit message: pcb changes v2
Parts:
- moved C31 0.55 mm to (139.7, 236.3)
Routing:
- net Net-(U2-SW): track 0.00 -> 7.91 mm
- net Net-(U3-SW): track 0.00 -> 7.84 mm
- net VCCOB0: track 47.4 -> 53.8 mm
- net MGTAVTT: track 8.13 -> 12.1 mm
- net +12V: track 2.95 -> 6.79 mm
- net Net-(U3-FB): track 0.00 -> 3.60 mm
- net VCCOB33: track 4.41 -> 7.92 mm
- net Net-(U4-ADJ/GND): track 0.31 -> 3.58 mm
- net Net-(U2-FB): track 0.00 -> 3.00 mm
- net Net-(U3-COMP): track 0.00 -> 2.03 mm
- net Net-(U2-COMP): track 0.00 -> 2.03 mm
- net Net-(U3-EN): track 0.00 -> 2.01 mm
- net Net-(U2-EN): track 0.00 -> 2.01 mm
- net Net-(U2-BS): track 0.00 -> 1.93 mm
- net Net-(U3-BS): track 0.00 -> 1.84 mm
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