File: hardware/arcticvideo.kicad_pcb (KiCad board)
At the start: 8 copper layers, 312 x 98.8 mm, 220 parts, among them J1 472720024, J2 Conn_Coaxial, J3 Conn_Coaxial, J5 Bus_PCI_Express_x4, U1 XC7A75T-FGG676, U10 TPS51200DRCR, U11 TPS62175DQCR, U12 PESD5V0L2BT, U13 AMS1117-ADJ, U2 MP2307DN-LF-Z, U3 MP2307DN-LF-Z, U4 AMS1117-ADJ, U5 AMS1117-1.8, U6 PESD5V0L2BT, U7 HD3SS215IRTQT, U8 MT25QL256ABA1EW7-0SIT, U9 MT41K256M16TW-107:P

Commit message: pcb things
Parts:
- added J4: Conn_ARM_JTAG_SWD_10, Connector_PinSocket_2.54mm:PinSocket_2x05_P2.54mm_Vertical, F.Cu at (146.7, 97.7)
- added SW1: SW_DIP_x08, Button_Switch_THT:SW_DIP_SPSTx08_Slide_9.78x22.5mm_W7.62mm_P2.54mm, F.Cu at (92.3, 170.6)
- C1, C10, C11, C12, C123, C124, C125, C126, C127, C128, C129, C13, C134, C14, C15, C16, C19, C2, C20, C23, C26, C27, C28, C29, C32, C33, C34, C35, C36, C37, C38, C39, C40, C41, C42, C43, C44, C45, C46, C47, C48, C49, C50, C51, C52, C53, C54, C55, C56, C57, C58, C59, C60, C61, C62, C63, C64, C65, C66, C67, C68, C69, C7, C70, C71, C72, C73, C74, C75, C76, C77, C78, C79, C8, C80, C81, C82, C83, C84, C85, C86, C87, C9, R11, R13, R16, R18, R20, R23, R24, R25, R26, R48, R49, R50, R51, R52, R53, R54, R56, R57, R58: moved to B.Cu
- moved C124 152.0 mm to (171.9, 137.7), turned to -90 degrees
- moved C125 148.4 mm to (166.3, 137.7), turned to -90 degrees
- moved C128 148.2 mm to (174.1, 137.7), turned to -90 degrees
- moved C123 147.1 mm to (167.4, 137.7), turned to -90 degrees
- moved C129 145.4 mm to (169.5, 137.7), turned to -90 degrees
- moved C126 145.4 mm to (173.0, 137.7), turned to -90 degrees
- moved C127 142.4 mm to (168.4, 137.7), turned to -90 degrees
- moved C11 131.5 mm to (173.9, 153.7), turned to 180 degrees
- moved C10 131.0 mm to (173.9, 152.7), turned to 180 degrees
- moved C9 130.4 mm to (173.9, 151.6), turned to 180 degrees
- moved C7 128.8 mm to (173.9, 150.6), turned to 180 degrees
- moved C76 127.3 mm to (182.7, 147.4), turned to 180 degrees
- moved C19 124.6 mm to (166.8, 145.8), turned to -90 degrees
- moved C73 124.4 mm to (182.7, 146.3), turned to 180 degrees
- moved C1 123.8 mm to (173.9, 148.5), turned to 180 degrees
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Connections:
- R24 pad 1: SW1_IN -> SW2_IN
Routing:
- net +12V: track 6.79 -> 209.3 mm, vias 0 -> 8
- net GND: track 9.00 -> 177.7 mm, vias 3 -> 147
- net (no net): track 0.00 -> 111.8 mm, vias 694 -> 69
- net VCCOB33: track 7.92 -> 93.4 mm, vias 0 -> 37
- net AUX_N: track 0.00 -> 78.4 mm, vias 0 -> 2
- net DA1_P: track 0.00 -> 75.1 mm, vias 0 -> 2
- net DA1_N: track 0.00 -> 75.1 mm, vias 0 -> 2
- net DA0_P: track 0.00 -> 73.0 mm, vias 0 -> 2
- net DA0_N: track 0.00 -> 72.9 mm, vias 0 -> 2
- net DB0_P: track 0.00 -> 72.7 mm, vias 0 -> 2
- net DB0_N: track 0.00 -> 72.6 mm, vias 0 -> 2
- net DB1_P: track 0.00 -> 72.6 mm, vias 0 -> 2
- net DB1_N: track 0.00 -> 72.5 mm, vias 0 -> 2
- net *RAS: track 0.00 -> 63.3 mm, vias 0 -> 3
- net A13: track 0.00 -> 57.6 mm, vias 0 -> 4
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Other:
- board text added: "U1"
- board text added: "XC7A75T-FGG676"

Commit message: finished pcb
Parts:
- added C134: 100n, Capacitor_SMD:C_0402_1005Metric, F.Cu at (111.5, 145.7)
- added C135: 100n, Capacitor_SMD:C_0402_1005Metric, F.Cu at (115.3, 147.2)
- added C136: 1u, Capacitor_SMD:C_0402_1005Metric, F.Cu at (111.5, 144.7)
- added C137: 1u, Capacitor_SMD:C_0402_1005Metric, F.Cu at (115.3, 148.3)
- added C138: 4.7u, Capacitor_SMD:C_0402_1005Metric, F.Cu at (111.5, 142.5)
- added C139: 4.7u, Capacitor_SMD:C_0402_1005Metric, F.Cu at (115.3, 150.5)
- added C140: 470n, Capacitor_SMD:C_0402_1005Metric, F.Cu at (108.4, 140.5)
- added C141: 470n, Capacitor_SMD:C_0402_1005Metric, F.Cu at (117.8, 152.5)
- added C142: 10u, Capacitor_SMD:C_0402_1005Metric, F.Cu at (108.5, 137.5)
- added C143: 10u, Capacitor_SMD:C_0402_1005Metric, F.Cu at (117.8, 155.5)
- added C144: 10u, Capacitor_SMD:C_0402_1005Metric, F.Cu at (107.4, 137.5)
- added C145: 10u, Capacitor_SMD:C_0402_1005Metric, F.Cu at (118.9, 155.5)
- added C146: 100n, Capacitor_SMD:C_0402_1005Metric, F.Cu at (118.7, 139.3)
- added C147: 100n, Capacitor_SMD:C_0402_1005Metric, F.Cu at (108.1, 153.8)
- added C148: 100n, Capacitor_SMD:C_0402_1005Metric, F.Cu at (118.7, 137.7)
- added C149: 100n, Capacitor_SMD:C_0402_1005Metric, F.Cu at (108.1, 155.3)
- added C150: 10u, Capacitor_SMD:C_0402_1005Metric, F.Cu at (112.5, 134.5)
- added C151: 100n, Capacitor_SMD:C_0402_1005Metric, F.Cu at (114.9, 135.6)
- added C152: 10u, Capacitor_SMD:C_0402_1005Metric, F.Cu at (114.3, 158.2)
- added C153: 100n, Capacitor_SMD:C_0402_1005Metric, F.Cu at (111.9, 157.4)
- added C154: 100n, Capacitor_SMD:C_0402_1005Metric, F.Cu at (114.9, 134.5)
- added C155: 100n, Capacitor_SMD:C_0402_1005Metric, F.Cu at (111.9, 158.5)
- added C156: 100n, Capacitor_SMD:C_0402_1005Metric, F.Cu at (114.9, 133.4)
- added C157: 100n, Capacitor_SMD:C_0402_1005Metric, F.Cu at (111.9, 159.6)
- added D7: LED, LED_SMD:LED_0402_1005Metric, B.Cu at (138.5, 100.5)
- added G***: LOGO-10mm, arcticvideo:LOGO-10mm, F.Cu at (109.4, 187.5)
- added H1: MountingHole_Pad, MountingHole:MountingHole_2.7mm_Pad_Via, F.Cu at (94.0, 193.0)
- added H2: MountingHole_Pad, MountingHole:MountingHole_3mm_Pad_Via, F.Cu at (94.3, 97.8)
- added IC1: GS12142, arcticvideo:QFN40P400X600X100-41N-D, F.Cu at (113.4, 139.1)
- added IC2: GS12142, arcticvideo:QFN40P400X600X100-41N-D, F.Cu at (113.4, 153.9)
- added R33: 1k, Resistor_SMD:R_0402_1005Metric, B.Cu at (138.5, 97.4)
- added R49: 100k, Resistor_SMD:R_0402_1005Metric, F.Cu at (114.3, 142.5)
- added R50: 100k, Resistor_SMD:R_0402_1005Metric, F.Cu at (114.3, 143.6)
- added R51: 100k, Resistor_SMD:R_0402_1005Metric, F.Cu at (112.5, 150.5)
- added R52: 100k, Resistor_SMD:R_0402_1005Metric, F.Cu at (112.5, 149.4)
- added R53: 2, Resistor_SMD:R_0402_1005Metric, F.Cu at (111.5, 143.6)
- added R54: 2, Resistor_SMD:R_0402_1005Metric, F.Cu at (115.3, 149.4)
- added R55: 100k, Resistor_SMD:R_0402_1005Metric, F.Cu at (116.9, 142.4)
- added R56: 100k, Resistor_SMD:R_0402_1005Metric, F.Cu at (110.0, 150.5)
- added R57: 100k, Resistor_SMD:R_0402_1005Metric, F.Cu at (106.2, 137.5)
- added R58: 100k, Resistor_SMD:R_0402_1005Metric, F.Cu at (120.0, 155.5)
- added R59: 100k, Resistor_SMD:R_0402_1005Metric, F.Cu at (112.5, 133.4)
- added R60: 100k, Resistor_SMD:R_0402_1005Metric, F.Cu at (114.3, 159.3)
- C12, C19, C27, C32, C33, C34, C35, C36, C67, C68, C69: footprint Capacitor_SMD:C_0402_1005Metric -> Capacitor_SMD:C_0603_1608Metric
- C92, C94: value 100n -> 4.7u
- R65: renamed from R53; moved to F.Cu
- moved C54 21.9 mm to (150.9, 156.9), turned to 0 degrees
- moved C32 21.5 mm to (159.6, 138.5), turned to -90 degrees
- moved C64 20.5 mm to (150.9, 155.8), turned to 0 degrees
- moved C37 20.0 mm to (158.4, 138.5), turned to -90 degrees
- moved C49 19.0 mm to (150.9, 154.7), turned to 0 degrees
- moved C42 18.6 mm to (157.3, 138.5), turned to -90 degrees
- moved C59 17.5 mm to (150.9, 153.6), turned to 0 degrees
- moved C57 17.2 mm to (156.2, 138.5), turned to -90 degrees
- moved C44 16.1 mm to (150.9, 152.5), turned to 0 degrees
- moved C47 15.9 mm to (155.1, 138.5), turned to -90 degrees
- moved C39 14.6 mm to (150.9, 151.4), turned to 0 degrees
- moved C62 14.6 mm to (154.0, 138.5), turned to -90 degrees
- moved C52 13.3 mm to (152.9, 138.5), turned to -90 degrees
- moved C34 13.1 mm to (150.9, 150.2), turned to 0 degrees
- moved C36 10.2 mm to (160.2, 170.1), turned to 90 degrees
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- renumbered C134 to C158, R33 to R34, R34 to R35, R35 to R36, R36 to R37, R37 to R38, R38 to R39, R39 to R40, R40 to R41, R41 to R42, R42 to R43, R43 to R44, R44 to R45, R45 to R46, R46 to R47, R47 to R48, R48 to R61, R49 to R62, R50 to R63, R51 to R64, R52 to R66, R55 to R67, R54 to R68, R56 to R69, R57 to R70, R58 to R71
Connections:
- R30 pad 2: SDI_1_MON -> LED_3
- R31 pad 2: SDI_2_MON -> LED_4
- R32 pad 2: EXTRA_MON -> LED_5
- U1 pad AC14: SDI_1 -> SDI_1_DDO0_P
- U1 pad AC8: SDI_1 -> unconnected-(U1E-MGTPTXP2_213-PadAC8)
- U1 pad AD14: SDI_2 -> SDI_1_DDO0_N
- U1 pad AD8: SDI_2 -> unconnected-(U1E-MGTPTXN2_213-PadAD8)
- U1 pad AE11: unconnected-(U1E-MGTPRXP3_213-PadAE11) -> SDI_2_DDO0_P
- U1 pad AF11: unconnected-(U1E-MGTPRXN3_213-PadAF11) -> SDI_2_DDO0_N
- U1 pad J14: unconnected-(U1B-IO_L2P_T0_AD8P_15-PadJ14) -> SDI_2_PLL
- U1 pad J15: unconnected-(U1B-IO_L2N_T0_AD8N_15-PadJ15) -> SDI_1_CS
- U1 pad J16: unconnected-(U1B-IO_L1N_T0_AD0N_15-PadJ16) -> SDI_2_LOS
- U1 pad J21: unconnected-(U1B-IO_L12N_T1_MRCC_15-PadJ21) -> SDI_2_SCLK
- U1 pad K15: unconnected-(U1B-IO_L1P_T0_AD0P_15-PadK15) -> SDI_1_PLL
- U1 pad K16: unconnected-(U1B-IO_L3P_T0_DQS_AD1P_15-PadK16) -> SDI_1_SDIN
- U1 pad K17: unconnected-(U1B-IO_L3N_T0_DQS_AD1N_15-PadK17) -> SDI_1_SDOUT
- U1 pad K18: unconnected-(U1B-IO_0_15-PadK18) -> SDI_1_LOS
- U1 pad K21: unconnected-(U1B-IO_L12P_T1_MRCC_15-PadK21) -> SDI_1_SCLK
- U1 pad L14: unconnected-(U1B-IO_L4N_T0_15-PadL14) -> SDI_2_SDIN
- U1 pad M14: unconnected-(U1B-IO_L4P_T0_15-PadM14) -> SDI_2_CS
- U1 pad M15: unconnected-(U1B-IO_L5P_T0_AD9P_15-PadM15) -> SDI_2_SDOUT
- U1 pad T15: SDI_1_MON -> unconnected-(U1A-IO_L20N_T3_13-PadT15)
- U1 pad U15: SDI_2_MON -> LED_5
- U1 pad U16: EXTRA_MON -> LED_6
- U1 pad V18: unconnected-(U1A-IO_L19P_T3_13-PadV18) -> LED_4
- U1 pad W19: unconnected-(U1A-IO_L18N_T2_13-PadW19) -> LED_3
Routing:
- net VCCOB0: track 98.6 -> 725.2 mm, vias 21 -> 46
- net GND: track 177.7 -> 598.6 mm, vias 147 -> 225
- net VCCAUX: track 25.5 -> 361.8 mm, vias 17 -> 34
- net VCCOB33: track 93.4 -> 351.5 mm, vias 37 -> 43
- net VCCADC: track 13.7 -> 262.9 mm, vias 18 -> 23
- net MGTAVTT: track 15.6 -> 207.6 mm, vias 12 -> 14
- net (no net): track 111.8 -> 0.00 mm, vias 69 -> 1
- net INIT_B_LED: track 0.71 -> 102.6 mm, vias 1 -> 3
- net SW4_OUT: track 0.71 -> 96.9 mm
- net SW5_OUT: track 0.71 -> 94.5 mm
- net LED_3: track 0.00 -> 90.4 mm, vias 0 -> 1
- net TDI: track 0.71 -> 89.7 mm, vias 1 -> 2
- net TMS: track 0.71 -> 83.0 mm
- net LED_6: track 0.00 -> 82.0 mm, vias 0 -> 1
- net LED_5: track 0.00 -> 79.8 mm, vias 0 -> 1
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Other:
- board size 312 x 98.8 mm -> 134.5 x 101.3 mm
