File: hardware/flashram.kicad_sch (KiCad schematic)
At the start: 24 parts, among them U10 TPS51200DRCR, U8 MT25QL256ABA1EW7-0SIT, U9 MT41K256M16TW-107:P

Commit message: pcb things
Changed lines of the file:
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@@
+	(wire
+		(pts
+			(xy 132.08 102.87) (xy 134.62 102.87)
+		)
+		(stroke
+			(width 0)
+			(type default)
+		)
+	)
 	(wire
 		(pts
@@
 	(wire
 		(pts
+			(xy 132.08 92.71) (xy 135.89 92.71)
+		)
+		(stroke
+			(width 0)
+			(type default)
+		)
+	)
+	(wire
+		(pts
 			(xy 151.13 120.65) (xy 151.13 85.09)
 		)
@@
 	(wire
 		(pts
+			(xy 132.08 133.35) (xy 138.43 133.35)
+		)
+		(stroke
+			(width 0)
+			(type default)
+		)
+	)
+	(wire
+		(pts
 			(xy 81.28 138.43) (xy 66.04 138.43)
 		)
@@
 	(wire
 		(pts
+			(xy 132.08 115.57) (xy 135.89 115.57)
+		)
+		(stroke
+			(width 0)
+			(type default)
+		)
+	)
+	(wire
+		(pts
 			(xy 68.58 118.11) (xy 68.58 120.65)
 		)
@@
 		)
 		(stroke
+			(width 0)
+			(type default)
+		)
+	)
+	(wire
+		(pts
+			(xy 132.08 146.05) (xy 135.89 146.05)
+		)
+		(stroke

Commit message: finished pcb
Parts:
- renumbered R33 to R34, R34 to R35, R35 to R36, R36 to R37, R37 to R38, R38 to R39

Commit message: added changed
Parts:
- C100, C101, C102, C103, C108, C98, C99: Arrow Price/Stock (none) -> $1.0332
- C104, C97: Arrow Price/Stock (none) -> $3.2704
- C105, C107, C109, C110, C111: Arrow Price/Stock (none) -> $1.9152
- C106: Arrow Price/Stock (none) -> $0.2300
- R34: Arrow Price/Stock (none) -> $0.0120
- R35, R36, R37, R38, R39: Arrow Price/Stock (none) -> $0.2552
- U10: Arrow Price/Stock (none) -> $1.0026
- U8: Arrow Price/Stock (none) -> $39.7010
- U9: Arrow Price/Stock (none) -> $47.1002
