File: hardware/fpga1.kicad_sch (KiCad schematic)
At the start: 13 parts, among them U1 XC7A75T-FGG676

Commit message: finished pcb
Parts:
- added C134, C135, C146, C147, C148, C149, C151, C153, C154, C155, C156, C157: 100n, Capacitor_SMD:C_0402_1005Metric, symbol Device:C
- added C136, C137: 1u, Capacitor_SMD:C_0402_1005Metric, symbol Device:C
- added C138, C139: 4.7u, Capacitor_SMD:C_0402_1005Metric, symbol Device:C
- added C140, C141: 470n, Capacitor_SMD:C_0402_1005Metric, symbol Device:C
- added C142, C143, C144, C145, C150, C152: 10u, Capacitor_SMD:C_0402_1005Metric, symbol Device:C
- added IC1, IC2: GS12142, arcticvideo:QFN40P400X600X100-41N-D, symbol arcticvideo:GS12142
- added R49, R50, R51, R52, R55, R56, R57, R58, R59, R60: 100k, Resistor_SMD:R_0402_1005Metric, symbol Device:R
- added R53, R54: 2, Resistor_SMD:R_0402_1005Metric, symbol Device:R
- renumbered C134 to C158, R48 to R61, R49 to R62, R50 to R63, R51 to R64, R53 to R65, R52 to R66, R55 to R67, R54 to R68, R56 to R69, R57 to R70, R58 to R71
Connections:
- net GND: now also C134.1, C135.1, C136.1, C137.1, C142.2, C143.2, C144.2, C145.2, C146.1, C147.1, C148.1, C149.1, C150.2, C151.1, C152.2, C153.1, C154.1, C155.1, C156.1, C157.1, IC1.1 (VEE_DDI_1), IC1.14 (VSS_1), IC1.15 (VSS_2), IC1.19 (VEE_CORE_1), IC1.21 (VEEO_1), IC1.28 (VEEO_2), IC1.31 (VEE_CORE_2), IC1.37 (VEE_CORE_3), IC1.38 (VEE_CORE_4), IC1.8 (VEE_DDI_2), IC2.1 (VEE_DDI_1), IC2.14 (VSS_1), IC2.15 (VSS_2), IC2.19 (VEE_CORE_1), IC2.21 (VEEO_1), IC2.28 (VEEO_2), IC2.31 (VEE_CORE_2), IC2.37 (VEE_CORE_3), IC2.38 (VEE_CORE_4), IC2.8 (VEE_DDI_2), R50.1, R52.1, R53.2, R54.2, R55.2, R56.2, R59.2, R60.2
- net SDI_1: now also IC2.2 (SDI); no longer U1.AC14 (MGTPRXP2_213), U1.AC8 (MGTPTXP2_213)
- net SDI_2: now also IC1.2 (SDI); no longer U1.AD14 (MGTPRXN2_213), U1.AD8 (MGTPTXN2_213)
- net SDI_2_DDO0_P: now reaches U1.AE11 (MGTPRXP3_213)
- net SDI_2_DDO0_P: now also IC1.27 (DDO0)
- net SDI_2_DDO0_N: now reaches U1.AF11 (MGTPRXN3_213)
- net SDI_2_DDO0_N: now also IC1.26 (~{DDO0})
- new net: C152.1, IC2.30 (VCO_FILT10)
- new net: IC1.33 (GPIO2), R59.1
- new net: C138.1, R53.1
- new net: C134.2, IC1.5 (TERM)
- new net: C142.1, IC1.34 (VCO_FILT)
- new net: IC1.36 (GPIO3), R57.2
- new net: C140.1, IC1.40 (LF-)
- new net: C140.2, IC1.39 (LF+)
- new net: C143.1, IC2.34 (VCO_FILT)
- new net: C139.1, R54.1
- new net: C139.2, IC2.3 (SDI_TERM)
- new net: IC2.36 (GPIO3), R58.2
- new net: IC2.33 (GPIO2), R60.1
- new net: C141.2, IC2.39 (LF+)
- new net: C141.1, IC2.40 (LF-)
- new net: C135.2, IC2.5 (TERM)
- new net: C138.2, IC1.3 (SDI_TERM)
- new net: C150.1, IC1.30 (VCO_FILT10)
- new net +1V8: C136.2, C137.2, C144.1, C145.1, C146.2, C147.2, C148.2, C149.2, C151.2, C153.2, C154.2, C155.2, C156.2, C157.2, IC1.16 (VDD), IC1.20 (VCCO1P8_1), IC1.24 (VCCO_1), IC1.25 (VCCO_0), IC1.29 (VCCO1P8_0), IC1.35 (VCC_CORE), IC1.4 (VCC_DDI), IC2.16 (VDD), IC2.20 (VCCO1P8_1), IC2.24 (VCCO_1), IC2.25 (VCCO_0), IC2.29 (VCCO1P8_0), IC2.35 (VCC_CORE), IC2.4 (VCC_DDI), R49.2, R51.2, R57.1, R58.1
- new net SDI_1_CS: IC2.10 (~{CS}), R51.1
- new net SDI_1_DDO0_N: IC2.26 (~{DDO0}), U1.AD14 (MGTPRXN2_213)
- new net SDI_1_DDO0_P: IC2.27 (DDO0), U1.AC14 (MGTPRXP2_213)
- new net SDI_1_LOS: IC2.17 (GPIO0)
- new net SDI_1_PLL: IC2.18 (GPIO1)
- new net SDI_1_SCLK: IC2.13 (SCLK), R56.1
- new net SDI_1_SDIN: IC2.11 (SDIN), R52.2
- new net SDI_1_SDOUT: IC2.12 (SDOUT)
- new net SDI_2_CS: IC1.10 (~{CS}), R49.1
- new net SDI_2_LOS: IC1.17 (GPIO0)
- new net SDI_2_PLL: IC1.18 (GPIO1)
- new net SDI_2_SCLK: IC1.13 (SCLK), R55.1
- new net SDI_2_SDIN: IC1.11 (SDIN), R50.2
- new net SDI_2_SDOUT: IC1.12 (SDOUT)
Other:
- moved on the sheet: C158, R61, R62, R63, R64, R65, R66, R67, R68, R69, R70, R71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

Commit message: added changed
Parts:
- C134, C135, C146, C147, C148, C149, C151, C153, C154, C155, C156, C157: Arrow Price/Stock (none) -> $0.2520
- C136, C137: Arrow Price/Stock (none) -> $0.5280
- C138, C139: Arrow Price/Stock (none) -> $3.2704
- C140, C141: Arrow Price/Stock (none) -> $0.7560
- C142, C143, C144, C145, C150, C152: Arrow Price/Stock (none) -> $1.9152
- C158: Arrow Price/Stock (none) -> $1.0332
- IC1, IC2: Arrow Price/Stock (none) -> $105.5416
- R49, R50, R51, R52, R55, R56, R57, R58, R59, R60: Arrow Price/Stock (none) -> $0.0640
- R53, R54: Arrow Price/Stock (none) -> $8.8676
- R61, R62, R64, R66, R68, R69, R70, R71: Arrow Price/Stock (none) -> $0.2552
- R63: Arrow Price/Stock (none) -> $0.0360
- R65, R67: Arrow Price/Stock (none) -> $0.0140
- U1: Arrow Price/Stock (none) -> $77.7344
