File: hardware/interfaces.kicad_sch (KiCad schematic)
At the start: 44 parts, among them J1 472720024, J2 Conn_Coaxial, J3 Conn_Coaxial, J4 Conn_ARM_JTAG_SWD_10, SW1 SW_DIP_x08, U6 PESD5V0L2BT, U7 HD3SS215IRTQT

Commit message: pcb things
Parts:
- J4: footprint (none) -> Connector_PinSocket_2.54mm:PinSocket_2x05_P2.54mm_Vertical
- SW1: footprint (none) -> Button_Switch_THT:SW_DIP_SPSTx08_Slide_9.78x22.5mm_W7.62mm_P2.54mm
Changed lines of the file:
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@@
 			)
 		)
-		(property "Footprint" ""
+		(property "Footprint" "Connector_PinSocket_2.54mm:PinSocket_2x05_P2.54mm_Vertical"
 			(at 250.19 41.91 0)
 			(hide yes)
@@
 			)
 		)
-		(property "Footprint" ""
+		(property "Footprint" "Button_Switch_THT:SW_DIP_SPSTx08_Slide_9.78x22.5mm_W7.62mm_P2.54mm"
 			(at 33.02 184.15 0)
 			(hide yes)

Commit message: finished pcb
Parts:
- added D7: LED, LED_SMD:LED_0402_1005Metric, symbol Device:LED
- added R33: 1k, Resistor_SMD:R_0402_1005Metric, symbol Device:R
- C92, C94: value 100n -> 4.7u
Connections:
- net GND: now also D7.1 (K)
- net SW1_IN: no longer R24.1
- net SW2_IN: now also R24.1
- net EXTRA_MON renamed LED_5
- net SDI_1_MON renamed LED_3
- net SDI_2_MON renamed LED_4
- new net: D7.2 (A), R33.1
- new net LED_6: R33.2

Commit message: added changed
Parts:
- C88, C89, C90, C91, C93, C95, C96: Arrow Price/Stock (none) -> $1.0332
- C92, C94: Arrow Price/Stock (none) -> $3.2704
- D1, D2, D3, D4, D5, D6, D7: Arrow Price/Stock (none) -> $0.6118
- J1: Arrow Price/Stock (none) -> $3.0170
- J2, J3: Arrow Price/Stock (none) -> $24.1028
- J4: now left out of the parts list
- R11, R14, R15, R16, R18, R20, R23, R24, R25, R26: Arrow Price/Stock (none) -> $0.2552
- R12, R19, R22: Arrow Price/Stock (none) -> $0.0320
- R13, R17: Arrow Price/Stock (none) -> $0.0640
- R21: Arrow Price/Stock (none) -> $0.0280
- R27, R28, R29, R30, R31, R32, R33: Arrow Price/Stock (none) -> $0.1000
- SW1: Arrow Price/Stock (none) -> $0.7663
- U6: Arrow Price/Stock (none) -> $0.3306
- U7: Arrow Price/Stock (none) -> $8.3696
